File: hw/AmigaKeyboardAdapters/StandAlone-Adapter/StandAlone-Adapter.sch (KiCad schematic (older format))
At the start: 60 parts, among them J1 RJ10, J2 Conn_02x03_Odd_Even, P1 CONN_01X02, Q1 BSS138, Q2 BSS138, Q3 BSS138, U1 AZ1117-3.3, U3 STM32F401RCTx

Commit message: Modified footprint of RJ10 (it was reversed)
Parts:
- C4, C5, C6, C7, C8, C9: symbol C -> C-RESCUE-StandAlone-Adapter
- D1, D2, D3, D4: symbol LED -> LED-RESCUE-StandAlone-Adapter
- Q1, Q2, Q3: symbol BSS138 -> BSS138-RESCUE-StandAlone-Adapter
- R1, R10, R11, R12, R13, R2, R4, R5, R6, R7, R8, R9: symbol R -> R-RESCUE-StandAlone-Adapter

Commit message: Revert "Modified footprint of RJ10 (it was reversed)"
This reverts commit 65f5b3a9598e76c611fb4c453a8e3fe395b7212b.
Parts:
- C4, C5, C6, C7, C8, C9: symbol C-RESCUE-StandAlone-Adapter -> C
- D1, D2, D3, D4: symbol LED-RESCUE-StandAlone-Adapter -> LED
- Q1, Q2, Q3: symbol BSS138-RESCUE-StandAlone-Adapter -> BSS138
- R1, R10, R11, R12, R13, R2, R4, R5, R6, R7, R8, R9: symbol R-RESCUE-StandAlone-Adapter -> R

Commit message: From Kicad 4 to Kicad 5
Parts:
- removed AMIGA_KEYBOARD1: CONN_01X05, Pin_Headers:Pin_Header_Angled_1x05, symbol CONN_01X05
- removed BOOT0, BOOT1, DEBUG1: CONN_01X03, Pin_Headers:Pin_Header_Straight_1x03, symbol CONN_01X03
- removed P1, TP1/1, USB_ID1: CONN_01X02, Pin_Headers:Pin_Header_Straight_1x02, symbol CONN_01X02
- removed POWER1, SWDIO/CLK1: CONN_01X04, Pin_Headers:Pin_Header_Angled_1x04, symbol CONN_01X04
- removed U3: STM32F401RCTx, Housings_QFP:LQFP-64_10x10mm_Pitch0.5mm, symbol STM32F401RCTx
- removed USB1: CONN_01x04, RetroBitLab:USB_A_UP, symbol CONN_01X04
- added J10, J4: Conn_01x04, Connector_PinHeader_2.54mm:PinHeader_1x04_P2.54mm_Horizontal, symbol Connector_Generic:Conn_01x04
- added J11, J8, J9: Conn_01x02, Connector_PinHeader_2.54mm:PinHeader_1x02_P2.54mm_Vertical, symbol Connector_Generic:Conn_01x02
- added J2, J6, J7: Conn_01x03, Connector_PinHeader_2.54mm:PinHeader_1x03_P2.54mm_Vertical, symbol Connector_Generic:Conn_01x03
- added J5: Conn_01x05, Connector_PinHeader_2.54mm:PinHeader_1x05_P2.54mm_Horizontal, symbol Connector_Generic:Conn_01x05
- added TP2: amigaWorkbench, RetroBitLab:amigaWorkBench1, symbol Connector:TestPoint
- added TP3: amigaLogo, RetroBitLab:amigaLogo_BW_31x12mm, symbol Connector:TestPoint
- added TP4: GNU-GPL, RetroBitLab:Symbol_GNU-GPL_SilkScreen_Small, symbol Connector:TestPoint
- added TP5: USBLOGO, RetroBitLab:USB_PLUG_15x15mm, symbol Connector:TestPoint
- added U2: STM32F401RBTx, Package_QFP:LQFP-64_10x10mm_P0.5mm, symbol AmigaComponents:STM32F401RBTx
- added USB1: USB_A, RetroBitLab:CUI_UJ2-AH-4-TH, symbol Connector:USB_A
- C1, C2: footprint Capacitors_Tantalum_SMD:TantalC_SizeA_EIA-3216_HandSoldering -> Capacitor_Tantalum_SMD:CP_EIA-3216-12_Kemet-S_Pad1.58x1.35mm_HandSolder; symbol CP1 -> StandAlone-Adapter-rescue:CP1
- C10: renamed from C6; footprint Capacitors_SMD:C_1206_HandSoldering -> Capacitor_SMD:C_1206_3216Metric_Pad1.33x1.80mm_HandSolder; symbol C -> StandAlone-Adapter-rescue:C
- C11: renamed from C7; footprint Capacitors_SMD:C_1206_HandSoldering -> Capacitor_SMD:C_1206_3216Metric_Pad1.33x1.80mm_HandSolder; symbol C -> StandAlone-Adapter-rescue:C
- C12: renamed from C8; footprint Capacitors_SMD:C_1206_HandSoldering -> Capacitor_SMD:C_1206_3216Metric_Pad1.33x1.80mm_HandSolder; symbol C -> StandAlone-Adapter-rescue:C
- C13: renamed from C9; footprint Capacitors_SMD:C_1206_HandSoldering -> Capacitor_SMD:C_1206_3216Metric_Pad1.33x1.80mm_HandSolder; symbol C -> StandAlone-Adapter-rescue:C
- C14, C3: footprint Capacitors_SMD:C_1206_HandSoldering -> Capacitor_SMD:C_1206_3216Metric_Pad1.33x1.80mm_HandSolder; symbol C_Small -> StandAlone-Adapter-rescue:C_Small
- C4: renamed from C10; footprint Capacitors_SMD:C_1206_HandSoldering -> Capacitor_SMD:C_1206_3216Metric_Pad1.33x1.80mm_HandSolder; symbol C_Small -> StandAlone-Adapter-rescue:C_Small
- C5: renamed from C11; footprint Capacitors_Tantalum_SMD:TantalC_SizeA_EIA-3216_HandSoldering -> Capacitor_Tantalum_SMD:CP_EIA-3216-18_Kemet-A_Pad1.58x1.35mm_HandSolder; symbol CP1_Small -> StandAlone-Adapter-rescue:CP1_Small
- C6: renamed from C12; footprint Capacitors_SMD:C_1206_HandSoldering -> Capacitor_SMD:C_1206_3216Metric_Pad1.33x1.80mm_HandSolder; symbol C_Small -> StandAlone-Adapter-rescue:C_Small
- C7: renamed from C13; footprint Capacitors_SMD:C_1206_HandSoldering -> Capacitor_SMD:C_1206_3216Metric_Pad1.33x1.80mm_HandSolder; symbol C_Small -> StandAlone-Adapter-rescue:C_Small
- C8: renamed from C4; footprint Capacitors_SMD:C_1206_HandSoldering -> Capacitor_SMD:C_1206_3216Metric_Pad1.33x1.80mm_HandSolder; symbol C -> StandAlone-Adapter-rescue:C
- C9: renamed from C5; footprint Capacitors_SMD:C_1206_HandSoldering -> Capacitor_SMD:C_1206_3216Metric_Pad1.33x1.80mm_HandSolder; symbol C -> StandAlone-Adapter-rescue:C
- D1, D4: footprint LEDs:LED_1206 -> LED_SMD:LED_1206_3216Metric_Pad1.42x1.75mm_HandSolder; symbol LED -> StandAlone-Adapter-rescue:LED
- D2: renamed from D3; footprint LEDs:LED_1206 -> LED_SMD:LED_1206_3216Metric_Pad1.42x1.75mm_HandSolder; symbol LED -> StandAlone-Adapter-rescue:LED
- D3: renamed from D2; footprint LEDs:LED_1206 -> LED_SMD:LED_1206_3216Metric_Pad1.42x1.75mm_HandSolder; symbol LED -> StandAlone-Adapter-rescue:LED
- EN1: footprint Pin_Headers:Pin_Header_Straight_1x02 -> Connector_PinHeader_2.54mm:PinHeader_1x02_P2.54mm_Vertical; symbol CONN_01X02 -> StandAlone-Adapter-rescue:CONN_01X02
- H1, H2, H3, H4: footprint Connect:1pin -> RetroBitLab:MountingHole; symbol CONN_01X01 -> StandAlone-Adapter-rescue:CONN_01X01
- J1: symbol RJ10 -> StandAlone-Adapter-rescue:RJ10
- J3: renamed from J2; symbol Conn_02x03_Odd_Even -> StandAlone-Adapter-rescue:Conn_02x03_Odd_Even
- Q1: footprint TO_SOT_Packages_SMD:SOT-23 -> Package_TO_SOT_SMD:SOT-23; symbol BSS138 -> StandAlone-Adapter-rescue:BSS138
- Q2: renamed from Q3; footprint TO_SOT_Packages_SMD:SOT-23 -> Package_TO_SOT_SMD:SOT-23; symbol BSS138 -> StandAlone-Adapter-rescue:BSS138
- Q3: renamed from Q2; footprint TO_SOT_Packages_SMD:SOT-23 -> Package_TO_SOT_SMD:SOT-23; symbol BSS138 -> StandAlone-Adapter-rescue:BSS138
- R1, R11: footprint Resistors_SMD:R_1206_HandSoldering -> Resistor_SMD:R_1206_3216Metric_Pad1.30x1.75mm_HandSolder; symbol R -> StandAlone-Adapter-rescue:R
- R10: renamed from R7; footprint Resistors_SMD:R_1206_HandSoldering -> Resistor_SMD:R_1206_3216Metric_Pad1.30x1.75mm_HandSolder; symbol R -> StandAlone-Adapter-rescue:R
- R12: renamed from R9; footprint Resistors_SMD:R_1206_HandSoldering -> Resistor_SMD:R_1206_3216Metric_Pad1.30x1.75mm_HandSolder; symbol R -> StandAlone-Adapter-rescue:R
- R13: renamed from R8; footprint Resistors_SMD:R_1206_HandSoldering -> Resistor_SMD:R_1206_3216Metric_Pad1.30x1.75mm_HandSolder; symbol R -> StandAlone-Adapter-rescue:R
- R14: renamed from R12; footprint Resistors_SMD:R_1206_HandSoldering -> Resistor_SMD:R_1206_3216Metric_Pad1.30x1.75mm_HandSolder; symbol R -> StandAlone-Adapter-rescue:R
- R15: renamed from R10; footprint Resistors_SMD:R_1206_HandSoldering -> Resistor_SMD:R_1206_3216Metric_Pad1.30x1.75mm_HandSolder; symbol R -> StandAlone-Adapter-rescue:R
- R16, R17: footprint Resistors_SMD:R_1206_HandSoldering -> Resistor_SMD:R_1206_3216Metric_Pad1.30x1.75mm_HandSolder; symbol R_Small -> StandAlone-Adapter-rescue:R_Small
- R2: renamed from R6; footprint Resistors_SMD:R_1206_HandSoldering -> Resistor_SMD:R_1206_3216Metric_Pad1.30x1.75mm_HandSolder; symbol R -> StandAlone-Adapter-rescue:R
- R3: renamed from R2; footprint Resistors_SMD:R_1206_HandSoldering -> Resistor_SMD:R_1206_3216Metric_Pad1.30x1.75mm_HandSolder; symbol R -> StandAlone-Adapter-rescue:R
- R4: renamed from R3; footprint Resistors_SMD:R_1206_HandSoldering -> Resistor_SMD:R_1206_3216Metric_Pad1.30x1.75mm_HandSolder; symbol R_Small -> StandAlone-Adapter-rescue:R_Small
- R5: renamed from R13; footprint Resistors_SMD:R_1206_HandSoldering -> Resistor_SMD:R_1206_3216Metric_Pad1.30x1.75mm_HandSolder; symbol R -> StandAlone-Adapter-rescue:R
- R6: renamed from R14; footprint Resistors_SMD:R_1206_HandSoldering -> Resistor_SMD:R_1206_3216Metric_Pad1.30x1.75mm_HandSolder; symbol R_Small -> StandAlone-Adapter-rescue:R_Small
- R7: renamed from R15; footprint Resistors_SMD:R_1206_HandSoldering -> Resistor_SMD:R_1206_3216Metric_Pad1.30x1.75mm_HandSolder; symbol R_Small -> StandAlone-Adapter-rescue:R_Small
- R8: renamed from R4; footprint Resistors_SMD:R_1206_HandSoldering -> Resistor_SMD:R_1206_3216Metric_Pad1.30x1.75mm_HandSolder; symbol R -> StandAlone-Adapter-rescue:R
- R9: renamed from R5; footprint Resistors_SMD:R_1206_HandSoldering -> Resistor_SMD:R_1206_3216Metric_Pad1.30x1.75mm_HandSolder; symbol R -> StandAlone-Adapter-rescue:R
- RESET1: symbol SW_PUSH -> StandAlone-Adapter-rescue:SW_PUSH
- TP1: footprint Wire_Pads:SolderWirePad_single_0-8mmDrill -> TestPoint:TestPoint_Pad_D2.0mm; symbol TEST_1P -> StandAlone-Adapter-rescue:TEST_1P
- U1: footprint TO_SOT_Packages_SMD:SOT-223 -> Package_TO_SOT_SMD:SOT-223; symbol AZ1117-3.3 -> StandAlone-Adapter-rescue:AZ1117-3.3
- XT1: symbol Crystal -> StandAlone-Adapter-rescue:Crystal
Connections:
- net BOOT0: now also J2.2 (Pin_2)
- net BOOT1: now also J6.2 (Pin_2)
- net GND: now also C14.1, J10.2 (Pin_2), J10.3 (Pin_3), J11.1 (Pin_1), J2.3 (Pin_3), J4.1 (Pin_1), J5.4 (Pin_4), J6.3 (Pin_3), J7.1 (Pin_1), J8.2 (Pin_2), U2.12 (VSSA), U2.18 (VSS), U2.31 (VSS), U2.47 (VSS), U2.63 (VSS), USB1.4 (GND), USB1.5 (Shield); no longer C14.2
- net KBD_3v3_CLOCK: now also U2.10 (PC2)
- net KBD_3v3_DATA: now also U2.11 (PC3)
- net KBD_3v3_RESET: now also U2.9 (PC1)
- net KBD_CLOCK: now also J5.1 (Pin_1)
- net KBD_DATA: now also J5.2 (Pin_2)
- net KBD_RESET: now also J8.1 (Pin_1)
- net NRST: now also U2.7 (NRST)
- net SWDCLK: now also J4.3 (Pin_3), U2.49 (PA14)
- net SWDIO: now also J4.2 (Pin_2), U2.46 (PA13)
- net TP1: now also J9.2 (Pin_2), U2.14 (PA0)
- net TP2: now also J9.1 (Pin_1), U2.15 (PA1)
- net UART_RX_TTL: now also J7.2 (Pin_2), U2.17 (PA3)
- net UART_TX_TTL: now also J7.3 (Pin_3), U2.16 (PA2)
- net USB_ID: now also J11.2 (Pin_2), U2.43 (PA10)
- net USB_N: now also U2.44 (PA11)
- net USB_P: now also U2.45 (PA12)
- net VCC: now also C14.2, J10.1 (Pin_1), J5.5 (Pin_5), USB1.1 (VBUS); no longer C14.1
- net VCC12V: now also J10.4 (Pin_4)
- net VCC3V3: now also J2.1 (Pin_1), J4.4 (Pin_4), J6.1 (Pin_1), U2.13 (VREF+), U2.19 (VDD), U2.32 (VDD), U2.48 (VDD), U2.64 (VDD)
- net at C8.1, XT1.1: now also U2.5 (PH0)
- net at C9.1, XT1.2: now also U2.6 (PH1)
- net at R17.2: now also USB1.2 (D-)
- net at R16.2: now also USB1.3 (D+)
- net at R7.2: now also U2.28 (PB2)
- net at C7.1: now also U2.30 (VCAP1)
- net at R6.1: now also U2.60 (BOOT0)
- no-connect marks 72 -> 44
Other:
- note added: "BOTH STM32F401RBT6 or STM32F401RCT6\ncan be used here. The first has 128k FLASH\nand the latter has 256K FLASH"
- note added: "SILKSCREEN LOGOS"
- moved on the sheet: C14, R16, R17

Commit message: Rigenerated
Parts:
- removed TP2: amigaWorkbench, RetroBitLab:amigaWorkBench1, symbol Connector:TestPoint
- removed TP3: amigaLogo, RetroBitLab:amigaLogo_BW_31x12mm, symbol Connector:TestPoint
- removed TP4: GNU-GPL, RetroBitLab:Symbol_GNU-GPL_SilkScreen_Small, symbol Connector:TestPoint
- removed TP5: USBLOGO, RetroBitLab:USB_PLUG_15x15mm, symbol Connector:TestPoint
- added LOGO1: USB, RetroBitLab:USB_PLUG_15x15mm, symbol AmigaComponents:LOGO
- added LOGO2: GPL, Symbol:KiCad-Logo2_12mm_SilkScreen, symbol AmigaComponents:LOGO
- added LOGO3: STALKER!, RetroBitLab:Symbol_GNU-GPL_SilkScreen_Small, symbol AmigaComponents:LOGO
Connections:
- no-connect marks 44 -> 41
Other:
- note removed: "SILKSCREEN LOGOS"
- moved on the sheet: C7
Changed lines of the file:
@@
 L StandAlone-Adapter-rescue:GND #PWR019
 U 1 1 5B89F643
-P 6500 4400
-F 0 "#PWR019" H 6500 4150 50  0001 C CNN
-F 1 "GND" H 6500 4250 50  0000 C CNN
-F 2 "" H 6500 4400 50  0001 C CNN
-F 3 "" H 6500 4400 50  0001 C CNN
-	1    6500 4400
+P 6500 4410
+F 0 "#PWR019" H 6500 4160 50  0001 C CNN
+F 1 "GND" H 6500 4260 50  0000 C CNN
+F 2 "" H 6500 4410 50  0001 C CNN
+F 3 "" H 6500 4410 50  0001 C CNN
+	1    6500 4410
 	1    0    0    -1
 $EndComp
@@
 L StandAlone-Adapter-rescue:GND #PWR01
 U 1 1 5BEA509B
-P 950 10500
-F 0 "#PWR01" H 950 10250 50  0001 C CNN
-F 1 "GND" H 950 10350 50  0000 C CNN
-F 2 "" H 950 10500 50  0001 C CNN
-F 3 "" H 950 10500 50  0001 C CNN
-	1    950  10500
+P 950 10300
+F 0 "#PWR01" H 950 10050 50  0001 C CNN
+F 1 "GND" H 950 10150 50  0000 C CNN
+F 2 "" H 950 10300 50  0001 C CNN
+F 3 "" H 950 10300 50  0001 C CNN
+	1    950  10300
 	1    0    0    -1
 $EndComp
@@
 Connection ~ 10100 4450
 Wire Wire Line
-	6500 4200 6500 4400
-Wire Wire Line
 	3000 5550 3000 5750
 Connection ~ 3000 6000
@@
 Wire Wire Line
 	1600 10300 950  10300
-Wire Wire Line
-	950  10300 950  10500
 Wire Wire Line
 	2100 10300 2500 10300
@@
 L StandAlone-Adapter-rescue:C_Small C7
 U 1 1 5CB3B205
-P 6800 4900
-F 0 "C7" H 6810 4970 50  0000 L CNN
-F 1 "4.7u" H 6810 4820 50  0000 L CNN
-F 2 "Capacitor_SMD:C_1206_3216Metric_Pad1.33x1.80mm_HandSolder" H 6800 4900 50  0001 C CNN
-F 3 "" H 6800 4900 50  0000 C CNN
-	1    6800 4900
+P 6800 4865
+F 0 "C7" H 6810 4935 50  0000 L CNN
+F 1 "4.7u" H 6810 4785 50  0000 L CNN
+F 2 "Capacitor_SMD:C_1206_3216Metric_Pad1.33x1.80mm_HandSolder" H 6800 4865 50  0001 C CNN
+F 3 "" H 6800 4865 50  0000 C CNN
+	1    6800 4865
 	-1   0    0    1
 $EndComp
@@
 L StandAlone-Adapter-rescue:GND #PWR020
 U 1 1 5CB3B2CE
-P 6800 4800
-F 0 "#PWR020" H 6800 4550 50  0001 C CNN
-F 1 "GND" H 6800 4650 50  0000 C CNN
-F 2 "" H 6800 4800 50  0001 C CNN
-F 3 "" H 6800 4800 50  0001 C CNN
-	1    6800 4800
+P 6800 4725
+F 0 "#PWR020" H 6800 4475 50  0001 C CNN
+F 1 "GND" H 6800 4575 50  0000 C CNN
+F 2 "" H 6800 4725 50  0001 C CNN
+F 3 "" H 6800 4725 50  0001 C CNN
+	1    6800 4725
 	-1   0    0    1
 $EndComp
-Wire Wire Line
-	6800 5000 7950 5000
 Text Label 7700 5100 0    39   ~ 0
 VDDA
@@
 	800  700  800  2000
 $Comp
-L Connector:TestPoint TP2
-U 1 1 60802EF8
-P 6300 9750
-F 0 "TP2" H 6400 9900 50  0000 L CNN
-F 1 "amigaWorkbench" H 6250 9650 50  0000 L CNN
-F 2 "RetroBitLab:amigaWorkBench1" H 6500 9750 50  0001 C CNN
-F 3 "~" H 6500 9750 50  0001 C CNN
-	1    6300 9750
-	1    0    0    -1
-$EndComp
-$Comp
-L Connector:TestPoint TP3
-U 1 1 6080444A
-P 7000 9750
-F 0 "TP3" H 7100 9900 50  0000 L CNN
-F 1 "amigaLogo" H 7000 9650 50  0000 L CNN
-F 2 "RetroBitLab:amigaLogo_BW_31x12mm" H 7200 9750 50  0001 C CNN
-F 3 "~" H 7200 9750 50  0001 C CNN
-	1    7000 9750
-	1    0    0    -1
-$EndComp
-$Comp
-L Connector:TestPoint TP4
-U 1 1 60804689
-P 7600 9750
-F 0 "TP4" H 7700 9900 50  0000 L CNN
-F 1 "GNU-GPL" H 7550 9650 50  0000 L CNN
-F 2 "RetroBitLab:Symbol_GNU-GPL_SilkScreen_Small" H 7800 9750 50  0001 C CNN
-F 3 "~" H 7800 9750 50  0001 C CNN
-	1    7600 9750
-	1    0    0    -1
-$EndComp
-NoConn ~ 7600 9750
-NoConn ~ 7000 9750
-NoConn ~ 6300 9750
-Wire Notes Line
-	6100 10250 8200 10250
-Wire Notes Line
-	8200 10250 8200 9050
-Wire Notes Line
-	8200 9050 6100 9050
-Wire Notes Line
-	6100 9050 6100 10250
-Text Notes 6150 9200 0    79   ~ 16
-SILKSCREEN LOGOS
-$Comp
 L Connector:USB_A USB1
 U 1 1 60798564
@@
 	1    0    0    -1
 $EndComp
-$Comp
-L Connector:TestPoint TP5
-U 1 1 60926773
-P 7650 9300
-F 0 "TP5" H 7750 9450 50  0000 L CNN
-F 1 "USBLOGO" H 7600 9200 50  0000 L CNN
-F 2 "RetroBitLab:USB_PLUG_15x15mm" H 7850 9300 50  0001 C CNN
-F 3 "~" H 7850 9300 50  0001 C CNN
-	1    7650 9300
-	1    0    0    -1
-$EndComp
 Text Notes 9450 7350 0    79   ~ 16
 BOTH STM32F401RBT6 or STM32F401RCT6\ncan be used here. The first has 128k FLASH\nand the latter has 256K FLASH
+Wire Wire Line
+	6800 5000 7950 5000
+Wire Wire Line
+	6800 4965 6800 5000
+Wire Wire Line
+	6800 4725 6800 4765
+Wire Wire Line
+	6500 4200 6500 4410
+$Comp
+L AmigaComponents:LOGO LOGO1
+U 1 1 6368B065
+P 6135 9240
+F 0 "LOGO1" H 6200 9330 59  0000 L CNN
+F 1 "USB" H 6200 9230 59  0000 L CNN
+F 2 "RetroBitLab:USB_PLUG_15x15mm" H 6135 9240 59  0001 C CNN
+F 3 "" H 6135 9240 59  0001 C CNN
+	1    6135 9240
+	1    0    0    -1
+$EndComp
+$Comp
+L AmigaComponents:LOGO LOGO2
+U 1 1 6368CBB3
+P 6570 9235
+F 0 "LOGO2" H 6630 9330 59  0000 L CNN
+F 1 "GPL" H 6635 9235 59  0000 L CNN
+F 2 "Symbol:KiCad-Logo2_12mm_SilkScreen" H 6570 9235 59  0001 C CNN
+F 3 "" H 6570 9235 59  0001 C CNN
+	1    6570 9235
+	1    0    0    -1
+$EndComp
+$Comp
+L AmigaComponents:LOGO LOGO3
+U 1 1 63696ADE
+P 6965 9200
+F 0 "LOGO3" H 7000 9300 59  0000 L CNN
+F 1 "STALKER!" H 7000 9150 59  0000 L CNN
+F 2 "RetroBitLab:Symbol_GNU-GPL_SilkScreen_Small" H 6965 9200 59  0001 C CNN
+F 3 "" H 6965 9200 59  0001 C CNN
+	1    6965 9200
+	1    0    0    -1
+$EndComp
 $EndSCHEMATC
